File: pcb_core/project.kicad_pcb (KiCad board)
At the start: 2 copper layers, 18.3 x 25.9 mm, 43 parts, among them IC1 SX1509QBIULTRT

Commit message: Update PCB with infos
Other:
- board text added: "I2C Addresses: {A1} {A0} L L 0x3E L H 0x3F H L 0x70 H H 0x71"
