File: pcb_core/project.kicad_sch (KiCad schematic)
At the start: 43 parts, among them IC1 SX1509QBIULTRT

Commit message: Update PCB with infos
Changed lines of the file:
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@@
+		)
+	)
+	(text_box "I2C Addresses: \n{A1} {A0}\nL L 0x3E\nL H 0x3F\nH L 0x70\nH H 0x71"
+		(exclude_from_sim no)
+		(at 20.32 24.13 0)
+		(size 17.78 13.97)
+		(stroke
+			(width 0)
+			(type default)
+		)
+		(fill
+			(type none)
+		)
+		(effects
+			(font
+				(size 1.27 1.27)
+			)
+			(justify left top)
 		)
 	)
