File: pcb_PCA9685/project.kicad_sch (KiCad schematic)
At the start: 37 parts, among them IC1 PCA9685PW,118

Commit message: Update PCB for PCA9685
Parts:
- removed J24, J25, J26, J27: ~, Castellated_Holes:Castellated_Hole02, symbol Connector_Generic:Conn_01x01
- removed JP1: SolderJumper_3_Open, Jumper:SolderJumper-3_P1.3mm_Open_RoundedPad1.0x1.5mm, symbol Jumper:SolderJumper_3_Open
- added JP1, JP2, JP3, JP4, JP5, JP6, JP7: SolderJumper_2_Open, Jumper:SolderJumper-2_P1.3mm_Open_TrianglePad1.0x1.5mm, symbol Jumper:SolderJumper_2_Open
Connections:
- net GND is gone; now on net +3.3V: J17.1 (Pin_1)
- net +3.3V: now also J19.1 (Pin_1), J23.1 (Pin_1), JP1.2 (B), JP2.2 (B), JP3.2 (B), JP4.2 (B), JP5.2 (B), JP6.2 (B), JP7.2 (B)
- net A0: now also JP1.1 (A)
- net A1: now also JP3.1 (A)
- net A2: now also JP4.1 (A); no longer J23.1 (Pin_1)
- net A3: now also JP5.1 (A)
- net A4: now also JP6.1 (A); no longer J19.1 (Pin_1)
- net A5: now also JP7.1 (A); no longer J20.1 (Pin_1)
- net GNDD: now also J20.1 (Pin_1)
- net at R4.2: now also R3.2, JP2.1 (A)
- net OSCIO: no longer names the net of IC1.25 (EXTCLK)
- no-connect marks 4 -> 5
Other:
- moved on the sheet: J17, J18, J30, R3, R4, RN1

Commit message: Remove connector on own side
Parts:
- removed J21, J22: ~, Castellated_Holes:Castellated_Hole02, symbol Connector_Generic:Conn_01x01
Changed lines of the file:
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@@
-		)
-	)
-	(label "+3.3V"
-		(at 210.82 64.77 180)
-		(fields_autoplaced yes)
-		(effects
-			(font
-				(size 1.27 1.27)
-			)
-			(justify right bottom)
 		)
 	)
@@
 		)
 	)
-	(label "GNDD"
-		(at 210.82 68.58 180)
-		(fields_autoplaced yes)
-		(effects
-			(font
-				(size 1.27 1.27)
-			)
-			(justify right bottom)
-		)
-	)
 	(label "SCL"
 		(at 210.82 34.29 180)
@@
 	)
 	(symbol
-		(lib_id "Connector_Generic:Conn_01x01")
-		(at 215.9 64.77 0)
-		(unit 1)
-		(exclude_from_sim no)
-		(in_bom yes)
-		(on_board yes)
-		(dnp no)
-		(property "Reference" "J21"
-			(at 218.186 64.77 0)
-			(effects
-				(font
-					(size 1.27 1.27)
-				)
-				(justify left)
-			)
-		)
-		(property "Value" "~"
-			(at 218.44 66.0399 0)
-			(effects
-				(font
-					(size 1.27 1.27)
-				)
-				(justify left)
-			)
-		)
-		(property "Footprint" "Castellated_Holes:Castellated_Hole02"
-			(at 215.9 64.77 0)
-			(effects
-				(font
-					(size 1.27 1.27)
-				)
-				(hide yes)
-			)
-		)
-		(property "Datasheet" "~"
-			(at 215.9 64.77 0)
-			(effects
-				(font
-					(size 1.27 1.27)
-				)
-				(hide yes)
-			)
-		)
-		(property "Description" "Generic connector, single row, 01x01, script generated (kicad-library-utils/schlib/autogen/connector/)"
-			(at 215.9 64.77 0)
-			(effects
-				(font
-					(size 1.27 1.27)
-				)
-				(hide yes)
-			)
-		)
-		(pin "1"
-		)
-		(instances
-			(project "project"
-				(path "/eaded386-8ef5-4822-a552-66b037180f01"
-					(reference "J21")
-					(unit 1)
-				)
-			)
-		)
-	)
-	(symbol
 		(lib_id "power:+3.3V")
 		(at 68.58 154.94 0)
@@
 					(unit 1)
 				)
-			)
-		)
-	)
-	(symbol
-		(lib_id "Connector_Generic:Conn_01x01")
-		(at 215.9 68.58 0)
-		(unit 1)
-		(exclude_from_sim no)
-		(in_bom yes)
-		(on_board yes)
-		(dnp no)
-		(property "Reference" "J22"
-			(at 218.186 68.58 0)
-			(effects
-				(font
-					(size 1.27 1.27)
-				)
-				(justify left)
-			)
-		)
-		(property "Value" "~"
-			(at 218.44 69.8499 0)
-			(effects
-				(font
-					(size 1.27 1.27)
-				)
-				(justify left)
-			)
-		)
-		(property "Footprint" "Castellated_Holes:Castellated_Hole02"
-			(at 215.9 68.58 0)
-			(effects
-				(font
-					(size 1.27 1.27)
-				)
-				(hide yes)
-			)
-		)
-		(property "Datasheet" "~"
-			(at 215.9 68.58 0)
-			(effects
-				(font
-					(size 1.27 1.27)
-				)
-				(hide yes)
-			)
-		)
-		(property "Description" "Generic connector, single row, 01x01, script generated (kicad-library-utils/schlib/autogen/connector/)"
-			(at 215.9 68.58 0)
-			(effects
-				(font
-					(size 1.27 1.27)
-				)
-				(hide yes)
-			)
-		)
-		(pin "1"
-		)
-		(instances
-			(project "project"
-				(path "/eaded386-8ef5-4822-a552-66b037180f01"
-					(reference "J22")
-					(unit 1)
-				)

Commit message: Replace resistor array throw single resistor for reducing vias dn easy component selection
Parts:
- removed RN1: YC248-JR-0710KL, library:YC248JR0710KL, symbol YC248-JR-0710KL:YC248-JR-0710KL
- added R2, R5, R6, R7, R8, R9: 10k, Resistor_SMD:R_0402_1005Metric_Pad0.72x0.64mm_HandSolder, symbol Device:R
- J1, J10, J11, J12, J13, J14, J15, J16, J17, J18, J19, J2, J20, J23, J28, J29, J3, J30, J4, J5, J6, J7, J8, J9: now left out of the parts list
Connections:
- net A0: now also R2.1
- net A1: now also R5.1
- net A2: now also R6.1
- net A3: now also R7.1
- net A4: now also R8.1
- net A5: now also R9.1
- net GNDD: now also R2.2, R5.2, R6.2, R7.2, R8.2, R9.2
- no-connect marks 5 -> 1
Other:
- moved on the sheet: J23, J30

Commit message: Correct some warnings and missing 3D step files
Parts:
- C1: AISLER_MPN (none) -> Capacitor, 10uF, 0402 SMD
- IC1: AISLER_MPN (none) -> PCA9685PW,118; LCSC# (none) -> C2678753
- R1, R2, R3, R4, R5, R6, R7, R8, R9: AISLER_MPN (none) -> Resistor, 10k, 0402 SMD

Commit message: Add revision number to PCB
Other:
- company: (none) -> Thomas Fanninger
- title: (none) -> Breakout board: IO-Expander based on PCA9685
Changed lines of the file:
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@@
 	(generator_version "8.0")
 	(paper "A4")
+	(title_block
+		(title "Breakout board: IO-Expander based on PCA9685")
+		(date "2024-06-09")
+		(rev "1")
+		(company "Thomas Fanninger")
+	)
 	(junction
 		(at 80.01 157.48)

Commit message: Correct kibot for four layer
Parts:
- IC1: LCSC# C2678753 -> C2678753
Changed lines of the file:
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@@
 			)
 		)
-		(property "LCSC#" " C2678753"
+		(property "LCSC#" "C2678753"
 			(at 41.91 48.26 0)
 			(effects

Commit message: Correct kibot for four layer
Parts:
- added T1, T2, T3, T4: Tab, PCM_kikit:Tab, symbol PCM_kikit:Tab
