File: pcb_SX1509/project.kicad_pcb (KiCad board)
At the start: 4 copper layers, 18.3 x 25.9 mm, 38 parts, among them IC1 SX1509QBIULTRT

Commit message: Add panelize
Parts:
- added REF**: Tab, kikit:Tab, F.Cu at (97.8, 104.4)
- added REF**: Tab, kikit:Tab, F.Cu at (113.5, 104.4)
- added REF**: Tab, kikit:Tab, F.Cu at (113.5, 78.0)
- added REF**: Tab, kikit:Tab, F.Cu at (97.8, 78.0)
