File: pcb_SX1509/project.kicad_pcb (KiCad board)
At the start: 4 copper layers, 18.3 x 25.9 mm, 42 parts, among them IC1 SX1509QBIULTRT

Commit message: Add revision number to PCB
Other:
- board text added: "Rev.: ${REVISION}"
Changed lines of the file:
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@@
 	)
 	(paper "A4")
+	(title_block
+		(title "Breakout board: IO-Expander based on SX1509")
+		(date "2024-06-09")
+		(rev "1")
+		(company "Thomas Fanninger")
+	)
 	(layers
 		(0 "F.Cu" signal)
@@
 			)
 			(justify left bottom mirror)
+		)
+	)
+	(gr_text "Rev.: ${REVISION}"
+		(at 112.014 103.378 0)
+		(layer "B.SilkS")
+		(effects
+			(font
+				(size 0.6 0.6)
+				(thickness 0.1)
+				(bold yes)
+			)
+			(justify left bottom mirror)
